File: 00-09_Projects/02_Sensors/02.05_NUTS/hardware/Undertray_Board.kicad_sch (KiCad schematic)
At the start: 2 parts

Commit message: Design review changes
Parts:
- added H3, H4: MountingHole_Pad, symbol Mechanical:MountingHole_Pad
Connections:
- net GND: now also H3.1, H4.1
Other:
- sheet Sensors renamed Sensors_I2C
- note added: "Mounting Holes"
- moved on the sheet: H1, H2

Commit message: Rev A layout done
Parts:
- H1, H2, H3, H4: footprint (none) -> MountingHole:MountingHole_3.2mm_M3_DIN965_Pad
Changed lines of the file:
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@@
 			)
 		)
-		(property "Footprint" ""
+		(property "Footprint" "MountingHole:MountingHole_3.2mm_M3_DIN965_Pad"
 			(at 232.41 57.15 0)
 			(hide yes)
@@
 			)
 		)
-		(property "Footprint" ""
+		(property "Footprint" "MountingHole:MountingHole_3.2mm_M3_DIN965_Pad"
 			(at 194.31 57.15 0)
 			(hide yes)
@@
 			)
 		)
-		(property "Footprint" ""
+		(property "Footprint" "MountingHole:MountingHole_3.2mm_M3_DIN965_Pad"
 			(at 232.41 36.83 0)
 			(hide yes)
@@
 			)
 		)
-		(property "Footprint" ""
+		(property "Footprint" "MountingHole:MountingHole_3.2mm_M3_DIN965_Pad"
 			(at 194.31 36.83 0)
 			(hide yes)
