File: 00-09_Projects/02_Sensors/02.05_NUTS/hardware/Undertray_Board.kicad_pcb (KiCad board)
At the start: 4 copper layers, 39.6 x 47.7 mm, 93 parts, among them J1 USB_C_Receptacle_USB2.0_16P, J3 Conn_01x04_Socket, J4 SHF-105-01-L-D-SM-K-TR, J5 Conn_01x06_Pin, SW1 450404015514, SW2 TL3301EF160QG, U1 SN65HVD230, U2 STM32F302C8Tx, U3 AP2210K-3.3TRG1, U4 VL53L4CDV0DH/1, U5 ASM330LHBTR, U7 74HC2G32DP, Y1 RH100-16.000-9-1010-TR

Commit message: Design review rev 1 changes
Parts:
- removed kibuzzard-6AC9A90D: G***, kibuzzard-6AC9A90D
- added kibuzzard-6ACEE03A: G***, kibuzzard-6ACEE03A, F.Cu at (150.3, 46.4)
- J4: value SHF-105-01-L-D-SM-K-TR -> SHF-107-01-L-D-SM; footprint Undertray FP:SAMTEC_SHF-105-01-L-D-SM-K-TR -> Undertray FP:SAMTEC_SHF-107-01-L-D-SM
- moved +5V 24.9 mm to (127.2, 78.3)
- moved C10 8.21 mm to (136.7, 64.6)
- moved +3V3 2.36 mm to (128.7, 52.5), turned to -90 degrees
- moved TSCL 0.40 mm to (137.3, 46.0), turned to -90 degrees
- moved G*** 0.20 mm to (143.6, 45.8)
- moved TSDA 0.18 mm to (133.7, 46.0)
- moved J4 0.17 mm to (134.3, 58.4)
- renumbered TP3 to +3V3, TP2 to +5V, TP1 to +VBUS, C6 to C10, C17 to C11, C18 to C12, C11 to C13, C10 to C14, C20 to C15, C19 to C16, C21 to C17, C12 to C18, C13 to C19, C14 to C20, C15 to C21, C16 to C22, C5 to C3, C3 to C4, C22 to C5, C4 to C6, C9 to C7, C7 to C9, D8 to D10, D10 to D11, D11 to D2, D2 to D3, D5 to D4, D3 to D5, D4 to D6, D9 to D8, D6 to D9, TP5 to ISCL, TP4 to ISDA, J3 to J2, J5 to J3, R4 to R1, R11 to R10, R6 to R11, R15 to R12, R17 to R13, R7 to R14, R8 to R15, R9 to R17, R10 to R18, R5 to R2, R13 to R3, R1 to R4, R2 to R5, R3 to R6, R19 to R7, R12 to R8, R14 to R9, TP7 to TSCL, TP6 to TSDA, U3 to U2, U2 to U3, U7 to U4, U4 to U6
Connections:
- J4 pad 10: NRST -> unconnected-(J4-Pad10)
Routing:
- net +5V: track 46.2 -> 24.0 mm, vias 1 -> 0
- net UART_RX: track 28.4 -> 25.7 mm
- net UART_TX: track 26.2 -> 23.7 mm
- net +3V3: track 86.8 -> 85.0 mm, vias 22 -> 19
- net +VBUS: track 52.1 -> 53.7 mm
- net ToF_SDA: track 39.7 -> 40.9 mm
- net GND: track 33.9 -> 32.8 mm, vias 51 -> 47
- net ToF_SCL: track 38.7 -> 39.7 mm

Commit message: Design review Rev 1 changes
Routing:
- net +VBUS: track 53.7 -> 55.1 mm
Changed lines of the file:
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@@
+	)
+	(segment
+		(start 157.3 81.0247)
+		(end 155.6357 79.3604)
+		(width 0.6)
+		(layer "B.Cu")
+		(net "+VBUS")
 	)
 	(segment
@@
 	)
 	(segment
-		(start 155.3 88)
-		(end 155.3 79.6961)
-		(width 0.6)
-		(layer "B.Cu")
-		(net "+VBUS")
-	)
-	(segment
 		(start 133.6 70.1)
 		(end 134.4 70.9)
-		(width 0.6)
-		(layer "B.Cu")
-		(net "+VBUS")
-	)
-	(segment
-		(start 155.2 88.1)
-		(end 155.3 88)
 		(width 0.6)
 		(layer "B.Cu")
@@
 	)
 	(segment
+		(start 155.4 88)
+		(end 157.3 86.1)
+		(width 0.6)
+		(layer "B.Cu")
+		(net "+VBUS")
+	)
+	(segment
 		(start 136.6 69.5)
 		(end 136.6 67.1)
@@
 	)
 	(segment
+		(start 155.2 88.1)
+		(end 155.3 88)
+		(width 0.6)
+		(layer "B.Cu")
+		(net "+VBUS")
+	)
+	(segment
 		(start 144.5 85.3)
 		(end 147.3 88.1)
@@
 	)
 	(segment
-		(start 155.3 79.6961)
-		(end 155.6357 79.3604)
+		(start 155.3 88)
+		(end 155.4 88)
 		(width 0.6)
 		(layer "B.Cu")
@@
 		(width 0.6)
 		(layer "B.Cu")
+		(net "+VBUS")
+	)
+	(segment
+		(start 157.3 86.1)
+		(end 157.3 81.0247)
+		(width 0.6)
+		(layer "B.Cu")

Commit message: last changes
Parts:
- added G***: LOGO, Undertray FP:kevin_signature, F.Cu at (152.5, 46.8)
- moved kibuzzard-6AC9A8CB 1.75 mm to (153.3, 43.8)
- moved kibuzzard-6ACEE03A 1.75 mm to (150.4, 44.6)
Connections:
- J2 pad 1: GND -> +VBUS
- J2 pad 2: +VBUS -> GND
Routing:
- net +VBUS: track 55.1 -> 57.6 mm

Commit message: final changes
Parts:
- moved kibuzzard-6AC9A8CB 0.76 mm to (153.2, 44.5)
- moved kibuzzard-6ACEE03A 0.76 mm to (150.3, 45.4)
- moved G*** 0.72 mm to (152.4, 47.5)
Routing:
- net GND: vias 47 -> 45
Changed lines of the file:
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@@
 	(footprint "kibuzzard-6AC9A8CB"
 		(layer "F.Cu")
-		(at 153.3 43.75)
+		(at 153.2 44.5)
 		(descr "Generated with KiBuzzard")
 		(tags "kb_params=eyJBbGlnbm1lbnRDaG9pY2UiOiAiQ2VudGVyIiwgIkNhcExlZnRDaG9pY2UiOiAiWyIsICJDYXBSaWdodENob2ljZSI6ICJdIiwgIkZvbnRDb21ib0JveCI6ICJVYnVudHVNb25vLUIiLCAiSGVpZ2h0Q3RybCI6IDAuNSwgIkxheWVyQ29tYm9Cb3giOiAiRi5TaWxrUyIsICJMaW5lU3BhY2luZ0N0cmwiOiAxLjAsICJNdWx0aUxpbmVUZXh0IjogIlVuZGVydHJheSBTZW5zb3IgQm9hcmQiLCAiUGFkZGluZ0JvdHRvbUN0cmwiOiAwLjgsICJQYWRkaW5nTGVmdEN0cmwiOiAzLjgsICJQYWRkaW5nUmlnaHRDdHJsIjogMy44LCAiUGFkZGluZ1RvcEN0cmwiOiAwLjgsICJXaWR0aEN0cmwiOiAwLjAsICJhZHZhbmNlZENoZWNrYm94IjogdHJ1ZSwgImlubGluZUZvcm1hdFRleHRib3giOiBmYWxzZSwgImxpbmVvdmVyU3R5bGVDaG9pY2UiOiAiU3F1YXJlIiwgImxpbmVvdmVyVGhpY2tuZXNzQ3RybCI6IDF9")
@@
 	(footprint "kibuzzard-6ACEE03A"
 		(layer "F.Cu")
-		(at 150.4 44.65)
+		(at 150.3 45.4)
 		(descr "Generated with KiBuzzard")
 		(tags "kb_params=eyJBbGlnbm1lbnRDaG9pY2UiOiAiQ2VudGVyIiwgIkNhcExlZnRDaG9pY2UiOiAiWyIsICJDYXBSaWdodENob2ljZSI6ICIvIiwgIkZvbnRDb21ib0JveCI6ICJVYnVudHVNb25vLUIiLCAiSGVpZ2h0Q3RybCI6IDAuNSwgIkxheWVyQ29tYm9Cb3giOiAiRi5TaWxrUyIsICJMaW5lU3BhY2luZ0N0cmwiOiAxLjAsICJNdWx0aUxpbmVUZXh0IjogIlJldiAxLjAiLCAiUGFkZGluZ0JvdHRvbUN0cmwiOiAwLjgsICJQYWRkaW5nTGVmdEN0cmwiOiAzLjgsICJQYWRkaW5nUmlnaHRDdHJsIjogMy44LCAiUGFkZGluZ1RvcEN0cmwiOiAwLjgsICJXaWR0aEN0cmwiOiAwLjAsICJhZHZhbmNlZENoZWNrYm94IjogdHJ1ZSwgImlubGluZUZvcm1hdFRleHRib3giOiBmYWxzZSwgImxpbmVvdmVyU3R5bGVDaG9pY2UiOiAiU3F1YXJlIiwgImxpbmVvdmVyVGhpY2tuZXNzQ3RybCI6IDF9")
@@
 	(footprint "Undertray FP:kevin_signature"
 		(layer "F.Cu")
-		(at 152.5 46.75)
+		(at 152.440054 47.465316)
 		(property "Reference" "G***"
 			(at 0 0 0)
@@
 	)
 	(via
-		(at 150.4 47.7)
-		(size 0.6)
-		(drill 0.3)
-		(layers "F.Cu" "B.Cu")
-		(free yes)
-		(net "GND")
-	)
-	(via
 		(at 149.8 75.1)
 		(size 0.6)
@@
 		(net "GND")
 	)
-	(via
-		(at 153.4 47.8)
-		(size 0.6)
-		(drill 0.3)
-		(layers "F.Cu" "B.Cu")
-		(free yes)
-		(net "GND")
-	)

Commit message: extra changes
Parts:
- removed kibuzzard-6ACEE03A: G***, kibuzzard-6ACEE03A
- added kibuzzard-6ACFF7B6: G***, kibuzzard-6ACFF7B6, F.Cu at (150.3, 45.4)
- added kibuzzard-6ACFF7BD: G***, kibuzzard-6ACFF7BD, F.Cu at (153.2, 45.4)
- moved G*** 1.08 mm to (151.8, 46.6)

Commit message: final changes
Parts:
- moved +5V 1.10 mm to (128.3, 78.3)
- moved +VBUS 0.71 mm to (155.3, 87.4)
- moved +3V3 0.59 mm to (128.5, 52.0)
Routing:
- net +VBUS: track 57.6 -> 56.7 mm
- net +5V: track 24.0 -> 23.3 mm
Changed lines of the file:
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@@
 	(footprint "TestPoint:TestPoint_THTPad_D1.5mm_Drill0.7mm"
 		(layer "F.Cu")
-		(at 128.7 52.55 -90)
+		(at 128.5 52 -90)
 		(descr "THT pad as test Point, diameter 1.5mm, hole diameter 0.7mm")
 		(tags "test point THT pad")
@@
 	(footprint "TestPoint:TestPoint_THTPad_D1.5mm_Drill0.7mm"
 		(layer "F.Cu")
-		(at 127.2 78.3)
+		(at 128.3 78.3)
 		(descr "THT pad as test Point, diameter 1.5mm, hole diameter 0.7mm")
 		(tags "test point THT pad")
 		(property "Reference" "+5V"
-			(at 2.55 0 0)
+			(at -1.9 0 90)
 			(layer "F.SilkS")
 			(effects
@@
 	(footprint "TestPoint:TestPoint_THTPad_D1.5mm_Drill0.7mm"
 		(layer "F.Cu")
-		(at 155.2 88.1)
+		(at 155.3 87.4)
 		(descr "THT pad as test Point, diameter 1.5mm, hole diameter 0.7mm")
 		(tags "test point THT pad")
 		(property "Reference" "+VBUS"
-			(at -0.4 -1.8 0)
+			(at -0.1 1.8 0)
 			(layer "F.SilkS")
 			(effects
@@
 	)
 	(segment
-		(start 155.3 85.85)
-		(end 155.3 88)
+		(start 155.3 87.4)
+		(end 146.6 87.4)
 		(width 0.6)
 		(layer "B.Cu")
@@
 	)
 	(segment
-		(start 147.3 88.1)
-		(end 155.2 88.1)
+		(start 154.15 77.846101)
+		(end 154.15 82.925)
 		(width 0.6)
 		(layer "B.Cu")
@@
 	)
 	(segment
+		(start 155.3 84.075)
+		(end 155.3 87.4)
+		(width 0.6)
+		(layer "B.Cu")
+		(net "+VBUS")
+	)
+	(segment
 		(start 133.6 70.1)
 		(end 134.4 70.9)
@@
 	)
 	(segment
-		(start 154.15 84.7)
-		(end 155.3 85.85)
-		(width 0.6)
-		(layer "B.Cu")
-		(net "+VBUS")
-	)
-	(segment
 		(start 136.6 69.5)
 		(end 136.6 67.1)
@@
 	)
 	(segment
-		(start 144.5 85.3)
-		(end 147.3 88.1)
-		(width 0.6)
-		(layer "B.Cu")
-		(net "+VBUS")
-	)
-	(segment
-		(start 155.3 88)
-		(end 155.2 88.1)
+		(start 154.15 82.925)
+		(end 155.3 84.075)
 		(width 0.6)
 		(layer "B.Cu")
@@
 	)
 	(segment
-		(start 133.6 66.9)
-		(end 133.6 70.1)
+		(start 146.6 87.4)
+		(end 144.5 85.3)
 		(width 0.6)
 		(layer "B.Cu")
@@
 	)
 	(segment
-		(start 154.15 77.846101)
-		(end 154.15 84.7)
+		(start 133.6 66.9)
+		(end 133.6 70.1)
 		(width 0.6)
 		(layer "B.Cu")
@@
 	)
 	(segment
-		(start 126.9 78)
-		(end 126.9 74.9625)
+		(start 128.3 77.1)
+		(end 126.8375 75.6375)
 		(width 0.6)
 		(layer "F.Cu")
@@
 	)
 	(segment
-		(start 127.2 78.3)
-		(end 126.9 78)
+		(start 128.3 78.3)
+		(end 128.3 77.1)
 		(width 0.6)
 		(layer "F.Cu")
@@
 	)
 	(segment
-		(start 126.9 74.9625)
+		(start 126.8375 75.6375)
 		(end 126.8375 74.9)
 		(width 0.6)
@@
 	)
 	(segment
-		(start 134.599999 79.32)
-		(end 134.599999 80.09142)
+		(start 130.3 78.3)
+		(end 128.3 78.3)
 		(width 0.6)
 		(layer "B.Cu")
@@
 	)
 	(segment
-		(start 134.612499 77.37)
-		(end 134.612499 79.3075)
+		(start 134.599999 79.32)
+		(end 134.599999 80.09142)
 		(width 0.6)
 		(layer "B.Cu")
@@
 	)
 	(segment
-		(start 130.3 78.3)
-		(end 127.2 78.3)
+		(start 134.612499 77.37)
+		(end 134.612499 79.3075)
 		(width 0.6)
 		(layer "B.Cu")

Commit message: extra changes
Parts:
- removed kibuzzard-6ACFF7BD: G***, kibuzzard-6ACFF7BD
- added kibuzzard-6ACFFC7D: G***, kibuzzard-6ACFFC7D, F.Cu at (152.5, 45.7)
- moved kibuzzard-6ACFF7B6 0.42 mm to (150.3, 44.9)
- moved kibuzzard-6AC9A8CB 0.40 mm to (153.2, 44.1)
- moved G*** 0.38 mm to (152.0, 46.9)

Commit message: extra changes
Parts:
- removed the G*** at (152.0, 46.9)
- added G***: LOGO, Undertray FP:kevin_signature_test, F.Cu at (152.3, 47.7)
