File: 00-09_Projects/02_Sensors/02.05_NUTS/hardware/Sensors.kicad_sch (KiCad schematic)
At the start: 16 parts, among them U4 VL53L4CDV0DH/1, U5 ASM330LHBTR

Commit message: Design review changes
Parts:
- added FB2: FerriteBead, symbol Device:FerriteBead
- added JP2: SolderJumper_2_Open, symbol Jumper:SolderJumper_2_Open
- added TP4: TP_IMU_SDA, symbol Connector:TestPoint
- added TP5: TP_IMU_SCL, symbol Connector:TestPoint
- added TP6: TP_ToF_SDA, symbol Connector:TestPoint
- added TP7: TP_ToF_SCL, symbol Connector:TestPoint
Connections:
- net +3.3V is gone; now on net +3V3: R10.2, R7.2, R8.2, R9.2
- net +3V3: now also FB2.2, JP2.1 (A); no longer U4.11 (AVDD)
- net IMU_SCL: now also TP5.1
- net IMU_SDA: now also TP4.1
- net ToF_SCL: now also TP7.1
- net ToF_SDA: now also TP6.1
- new net: FB2.1, JP2.2 (B), U4.11 (AVDD)
Other:
- note added: "I2C Testpoints"

Commit message: Rev A layout done
Parts:
- D10: footprint (none) -> LED_SMD:LED_Cree-PLCC4_3.2x2.8mm_CCW
- FB2: footprint (none) -> Inductor_SMD:L_0402_1005Metric_Pad0.77x0.64mm_HandSolder
- JP2: footprint (none) -> Jumper:SolderJumper-2_P1.3mm_Open_TrianglePad1.0x1.5mm
- TP4, TP5, TP6, TP7: footprint (none) -> TestPoint:TestPoint_THTPad_D1.5mm_Drill0.7mm
- U4: footprint LGA12_STM -> Undertray FP:LGA12_STM
- U5: footprint LGA-14L_2p5x3-0p5_STM -> Undertray FP:LGA-14L_2p5x3-0p5_STM-M
Connections:
- net +3V3: now also JP2.2 (B); no longer JP2.1 (A)
- net at FB2.1, U4.11 (AVDD): now also JP2.1 (A); no longer JP2.2 (B)
Other:
- moved on the sheet: JP2
Changed lines of the file:
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@@
 	(rectangle
 		(start 17.78 153.67)
-		(end 80.01 184.15)
+		(end 67.31 184.15)
 		(stroke
 			(width 0)
@@
 			)
 		)
-		(property "Footprint" ""
+		(property "Footprint" "TestPoint:TestPoint_THTPad_D1.5mm_Drill0.7mm"
 			(at 26.67 162.56 0)
 			(hide yes)
@@
 	(symbol
 		(lib_id "Jumper:SolderJumper_2_Open")
-		(at 116.84 45.72 180)
+		(at 116.84 45.72 0)
+		(mirror x)
 		(unit 1)
 		(body_style 1)
@@
 		(dnp no)
 		(property "Reference" "JP2"
-			(at 116.586 42.926 0)
+			(at 117.094 42.926 0)
 			(show_name no)
 			(do_not_autoplace no)
@@
 		)
 		(property "Value" "SolderJumper_2_Open"
-			(at 116.586 40.386 0)
+			(at 117.094 40.386 0)
 			(show_name no)
 			(do_not_autoplace no)
@@
 			)
 		)
-		(property "Footprint" ""
+		(property "Footprint" "Jumper:SolderJumper-2_P1.3mm_Open_TrianglePad1.0x1.5mm"
 			(at 116.84 45.72 0)
 			(hide yes)
@@
 			)
 		)
-		(property "Footprint" ""
+		(property "Footprint" "TestPoint:TestPoint_THTPad_D1.5mm_Drill0.7mm"
 			(at 26.67 170.18 0)
 			(hide yes)
@@
 			)
 		)
-		(property "Footprint" ""
+		(property "Footprint" "TestPoint:TestPoint_THTPad_D1.5mm_Drill0.7mm"
 			(at 48.26 162.56 0)
 			(hide yes)
@@
 			)
 		)
-		(property "Footprint" "LGA12_STM"
+		(property "Footprint" "Undertray FP:LGA12_STM"
 			(at 46.99 49.53 0)
 			(hide yes)
@@
 			)
 		)
-		(property "Footprint" ""
+		(property "Footprint" "LED_SMD:LED_Cree-PLCC4_3.2x2.8mm_CCW"
 			(at 115.57 113.03 0)
 			(hide yes)
@@
 			)
 		)
-		(property "Footprint" "LGA-14L_2p5x3-0p5_STM"
+		(property "Footprint" "Undertray FP:LGA-14L_2p5x3-0p5_STM-M"
 			(at 160.02 44.45 0)
 			(hide yes)
@@
 			)
 		)
-		(property "Footprint" ""
+		(property "Footprint" "TestPoint:TestPoint_THTPad_D1.5mm_Drill0.7mm"
 			(at 48.26 170.18 0)
 			(hide yes)
@@
 			)
 		)
-		(property "Footprint" ""
+		(property "Footprint" "Inductor_SMD:L_0402_1005Metric_Pad0.77x0.64mm_HandSolder"
 			(at 116.84 53.848 90)
 			(hide yes)

Commit message: Design review rev 1 changes
Parts:
- renumbered C12 to C18, C13 to C19, C14 to C20, C15 to C21, C16 to C22, D10 to D11, R6 to R11, R15 to R12, R17 to R13, R7 to R14, R8 to R15, R9 to R17, R10 to R18, TP6 to TP5, TP5 to TP6, U4 to U6

Commit message: extra changes
Parts:
- R12: value 100 -> 200
- R13, R16: value 22 -> 47
Changed lines of the file:
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@@
 			)
 		)
-		(property "Value" "22"
+		(property "Value" "47"
 			(at 102.87 111.76 90)
 			(show_name no)
@@
 			)
 		)
-		(property "Value" "100"
+		(property "Value" "200"
 			(at 102.87 106.68 90)
 			(show_name no)
@@
 			)
 		)
-		(property "Value" "22"
+		(property "Value" "47"
 			(at 102.87 116.84 90)
 			(show_name no)
