File: 00-09_Projects/02_Sensors/02.05_NUTS/hardware/mcu.kicad_sch (KiCad schematic)
At the start: 25 parts, among them SW1 SW_Nidec_CAS-120A1, SW2 SW_Push, U2 STM32F302C8Tx, U6 74HC2G32DP, Y1 RH100-16.000-9-1010-TR

Commit message: Design review changes
Parts:
- removed R13: 10k, Resistor_SMD:R_0603_1608Metric_Pad0.98x0.95mm_HandSolder, symbol Device:R
- removed U6: 74HC2G32DP, symbol 74xGxx:74AHC1G32
- added J4: Cortex Debug Header, symbol Connector_Generic:Conn_02x05_Odd_Even
- added JP1: SolderJumper_2_Open, symbol Jumper:SolderJumper_2_Open
- added R19: 220, symbol Device:R
- added U7: 74HC2G32DP, symbol 74xGxx:74AUC2G32
- D7, D8: value PESD3V3S1UL -> ACPDQC3V3T-HF
- SW1: value SW_Nidec_CAS-120A1 -> OS102011MA1QN1
Connections:
- net +3V3: now also JP1.2 (B), U7.8 (VCC)
- net +3V3A: now also JP1.1 (A)
- net BOOT0: now also U7.7
- net BOOT0_SW: now also U7.1
- net BOOT0_TRIG: now also U2.40 (PB4), U7.2; no longer U2.41 (PB5)
- net GND: now also J4.3 (Pin_3), J4.5 (Pin_5), J4.9 (Pin_9), U7.4 (GND)
- net NRST: now also J4.10 (Pin_10)
- net RCC_OSC_OUT: now also R19.2; no longer C18.1, Y1.3
- net SWCLK: now also J4.4 (Pin_4)
- net SWDIO: now also J4.2 (Pin_2)
- net ToF_LED_B: now also U2.19 (PB1); no longer U2.38 (PA15)
- net ToF_LED_G: now also U2.18 (PB0); no longer U2.39 (PB3)
- net ToF_LED_R: now also U2.17 (PA7); no longer U2.40 (PB4)
- new net: C18.1, R19.1, Y1.3
- new net CAN_SLEEP: U2.41 (PB5)
- new net SWO: J4.6 (Pin_6)
- new net VCC: J4.1 (Pin_1)
- no-connect marks 21 -> 25
Other:
- note added: "Cortex Debug"
- moved on the sheet: C20, D6, D9, FB1, R11, R14, SW1

Commit message: Rev A layout done
Parts:
- added J5: Conn_01x06_Pin, Connector_PinHeader_2.54mm:PinHeader_1x06_P2.54mm_Vertical, symbol Connector:Conn_01x06_Pin
- D7, D8: footprint (none) -> Diode_SMD:D_0402_1005Metric_Pad0.77x0.64mm_HandSolder
- FB1: footprint (none) -> Inductor_SMD:L_0402_1005Metric_Pad0.77x0.64mm_HandSolder
- J4: value Cortex Debug Header -> SHF-105-01-L-D-SM-K-TR; footprint (none) -> Undertray FP:SAMTEC_SHF-105-01-L-D-SM-K-TR
- JP1: footprint (none) -> Jumper:SolderJumper-2_P1.3mm_Open_TrianglePad1.0x1.5mm
- R19: footprint (none) -> Resistor_SMD:R_0603_1608Metric_Pad0.98x0.95mm_HandSolder
- SW1: value OS102011MA1QN1 -> 450404015514; footprint (none) -> Undertray FP:WS-SLSU_6p7x2p7_WRE
- SW2: value SW_Push -> TL3301EF160QG; footprint (none) -> Button_Switch_SMD:SW_Push_1P1T_NO_CK_KSC6xxG
- U7: footprint (none) -> Package_SO:TSSOP-8_3x3mm_P0.65mm
- Y1: footprint (none) -> Crystal:Crystal_SMD_WE_CFPX-180-4Pin_3.2x2.5mm
Connections:
- net VCC is gone; now on net +3V3: J4.1 (Pin_1)
- net BOOT0_TRIG: now also U2.39 (PB3); no longer U2.40 (PB4)
- net GND: now also SW1.4 (MP), SW1.5 (MP), SW1.6 (MP), SW1.7 (MP), J5.3 (Pin_3), J5.4 (Pin_4)
- net IMU_SCL: now also U2.42 (PB6); no longer U2.30 (PA9)
- net IMU_SDA: now also U2.43 (PB7); no longer U2.31 (PA10)
- net SWCLK: now also U2.37 (PA14); no longer U2.27 (PB14)
- net SWDIO: now also U2.34 (PA13); no longer U2.26 (PB13)
- net ToF_LED_B: now also U2.17 (PA7); no longer U2.19 (PB1)
- net ToF_LED_R: now also U2.19 (PB1); no longer U2.17 (PA7)
- net ToF_SCL: now also U2.30 (PA9); no longer U2.42 (PB6)
- net ToF_SDA: now also U2.31 (PA10); no longer U2.43 (PB7)
- net UART_TX: now reaches U2.21 (PB10)
- net UART_TX: now also J5.5 (Pin_5)
- net UART_RX: now reaches U2.22 (PB11)
- net UART_RX: now also J5.6 (Pin_6)
- net SWO: no longer names the net of J4.6 (Pin_6)
- new net CAN_H: J5.1 (Pin_1)
- new net CAN_L: J5.2 (Pin_2)
- no-connect marks 25 -> 24
Other:
- note added: "Debug Header Pins"
- moved on the sheet: C21, D7, D8, D9, R14, SW2, U7B

Commit message: Design review rev 1 changes
Parts:
- removed J4: SHF-105-01-L-D-SM-K-TR, Undertray FP:SAMTEC_SHF-105-01-L-D-SM-K-TR, symbol Connector_Generic:Conn_02x05_Odd_Even
- added J4: SHF-107-01-L-D-SM, Undertray FP:SAMTEC_SHF-107-01-L-D-SM, symbol Undertray_Board_sym:SHF-107-01-L-D-SM
- renumbered C6 to C10, C17 to C11, C18 to C12, C11 to C13, C10 to C14, C20 to C15, C19 to C16, C21 to C17, C9 to C7, C7 to C9, D8 to D10, D9 to D8, D6 to D9, J5 to J3, R11 to R10, R19 to R7, R12 to R8, R14 to R9, U2 to U3, U7 to U4
Connections:
- net +3V3: now also J4.03
- net GND: now also J4.05, J4.07, J4.11
- net NRST: now also J4.12
- net SWCLK: now also J4.06
- net SWDIO: now also J4.04
- new net SWO: J4.08
- no-connect marks 24 -> 27
Other:
- moved on the sheet: J3

Commit message: extra changes
Parts:
- added C23: 0.1uF, Capacitor_SMD:C_0603_1608Metric_Pad1.08x0.95mm_HandSolder, symbol Device:C
- added R19: 47k, Resistor_SMD:R_0402_1005Metric_Pad0.72x0.64mm_HandSolder, symbol Device:R
Connections:
- net BOOT0_TRIG: now also R19.1; no longer U4.2
- net GND: now also C23.2
- new net: C23.1, R19.2, U4.2
Other:
- moved on the sheet: D9, R10, U4A, U4B

Commit message: extra changes
Parts:
- R10, R9: value 220 -> 330
Connections:
- net SWO: no longer names the net of J4.08
- no-connect marks 27 -> 28
Changed lines of the file:
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@@
 	)
 	(no_connect
+		(at 52.07 171.45)
+	)
+	(no_connect
 		(at 85.09 58.42)
 	)
@@
 	(wire
 		(pts
+			(xy 19.05 165.1) (xy 19.05 166.37)
+		)
+		(stroke
+			(width 0)
+			(type default)
+		)
+	)
+	(wire
+		(pts
 			(xy 137.16 36.83) (xy 137.16 38.1)
 		)
@@
 	(wire
 		(pts
+			(xy 19.05 166.37) (xy 26.67 166.37)
+		)
+		(stroke
+			(width 0)
+			(type default)
+		)
+	)
+	(wire
+		(pts
 			(xy 218.44 36.83) (xy 218.44 38.1)
 		)
@@
 		)
 	)
-	(global_label "+3V3"
-		(shape input)
-		(at 26.67 166.37 180)
-		(fields_autoplaced yes)
-		(effects
-			(font
-				(size 1.27 1.27)
-			)
-			(justify right)
-		)
-		(property "Intersheetrefs" "${INTERSHEET_REFS}"
-			(at 18.6048 166.37 0)
-			(hide yes)
-			(show_name no)
-			(do_not_autoplace no)
-			(effects
-				(font
-					(size 1.27 1.27)
-				)
-				(justify right)
-			)
-		)
-	)
 	(global_label "NRST"
 		(shape input)
@@
 		)
 	)
-	(global_label "SWO"
-		(shape input)
-		(at 52.07 171.45 0)
-		(fields_autoplaced yes)
-		(effects
-			(font
-				(size 1.27 1.27)
-			)
-			(justify left)
-		)
-		(property "Intersheetrefs" "${INTERSHEET_REFS}"
-			(at 59.0466 171.45 0)
-			(hide yes)
-			(show_name no)
-			(do_not_autoplace no)
-			(effects
-				(font
-					(size 1.27 1.27)
-				)
-				(justify left)
-			)
-		)
-	)
 	(global_label "BOOT0_SW"
 		(shape input)
@@
 			)
 		)
-		(property "Value" "220"
+		(property "Value" "330"
 			(at 234.95 137.1599 0)
 			(show_name no)
@@
 	)
 	(symbol
+		(lib_id "power:+3V3")
+		(at 19.05 165.1 0)
+		(unit 1)
+		(body_style 1)
+		(exclude_from_sim no)
+		(in_bom yes)
+		(on_board yes)
+		(in_pos_files yes)
+		(dnp no)
+		(fields_autoplaced yes)
+		(property "Reference" "#PWR061"
+			(at 19.05 168.91 0)
+			(hide yes)
+			(show_name no)
+			(do_not_autoplace no)
+			(effects
+				(font
+					(size 1.27 1.27)
+				)
+			)
+		)
+		(property "Value" "+3V3"
+			(at 19.05 160.02 0)
+			(show_name no)
+			(do_not_autoplace no)
+			(effects
+				(font
+					(size 1.27 1.27)
+				)
+			)
+		)
+		(property "Footprint" ""
+			(at 19.05 165.1 0)
+			(hide yes)
+			(show_name no)
+			(do_not_autoplace no)
+			(effects
+				(font
+					(size 1.27 1.27)
+				)
+			)
+		)
+		(property "Datasheet" ""
+			(at 19.05 165.1 0)
+			(hide yes)
+			(show_name no)
+			(do_not_autoplace no)
+			(effects
+				(font
+					(size 1.27 1.27)
+				)
+			)
+		)
+		(property "Description" "Power symbol creates a global label with name \"+3V3\""
+			(at 19.05 165.1 0)
+			(hide yes)
+			(show_name no)
+			(do_not_autoplace no)
+			(effects
+				(font
+					(size 1.27 1.27)
+				)
+			)
+		)
+		(pin "1"
+		)
+		(instances
+			(project "Undertray_Board"
+				(path "/85866aa8-1074-44e2-a4f8-fc50fec0cbab/74cdce65-3117-4a3b-a9a5-a5d0459f2000"
+					(reference "#PWR061")
+					(unit 1)
+				)
+			)
+		)
+	)
+	(symbol
 		(lib_id "Device:C")
 		(at 218.44 41.91 0)
@@
 			)
 		)
-		(property "Value" "220"
+		(property "Value" "330"
 			(at 142.24 130.8099 0)
 			(show_name no)

Commit message: solder jumper for reset
Parts:
- added JP3: SolderJumper_2_Open, Jumper:SolderJumper-2_P1.3mm_Open_TrianglePad1.0x1.5mm, symbol Jumper:SolderJumper_2_Open
Connections:
- net BOOT0: now also JP3.1 (A)
- net BOOT0_SW: now also JP3.2 (B)
Changed lines of the file:
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@@
 	)
 	(junction
+		(at 199.39 118.11)
+		(diameter 0)
+		(color 0 0 0 0)
+	)
+	(junction
 		(at 139.7 67.31)
 		(diameter 0)
@@
 	(wire
 		(pts
+			(xy 232.41 107.95) (xy 232.41 120.65)
+		)
+		(stroke
+			(width 0)
+			(type default)
+		)
+	)
+	(wire
+		(pts
+			(xy 215.9 107.95) (xy 232.41 107.95)
+		)
+		(stroke
+			(width 0)
+			(type default)
+		)
+	)
+	(wire
+		(pts
 			(xy 195.58 36.83) (xy 203.2 36.83)
 		)
@@
 	(wire
 		(pts
+			(xy 199.39 118.11) (xy 199.39 107.95)
+		)
+		(stroke
+			(width 0)
+			(type default)
+		)
+	)
+	(wire
+		(pts
 			(xy 200.66 123.19) (xy 200.66 125.73)
 		)
@@
 	(wire
 		(pts
-			(xy 190.5 118.11) (xy 201.93 118.11)
+			(xy 190.5 118.11) (xy 199.39 118.11)
 		)
 		(stroke
@@
 	(wire
 		(pts
+			(xy 199.39 107.95) (xy 205.74 107.95)
+		)
+		(stroke
+			(width 0)
+			(type default)
+		)
+	)
+	(wire
+		(pts
 			(xy 127 67.31) (xy 139.7 67.31)
 		)
@@
 	(wire
 		(pts
+			(xy 199.39 118.11) (xy 201.93 118.11)
+		)
+		(stroke
+			(width 0)
+			(type default)
+		)
+	)
+	(wire
+		(pts
 			(xy 190.5 123.19) (xy 191.77 123.19)
 		)
@@
 					(unit 1)
 				)
+			)
+		)
+	)
+	(symbol
+		(lib_id "Jumper:SolderJumper_2_Open")
+		(at 210.82 107.95 180)
+		(unit 1)
+		(body_style 1)
+		(exclude_from_sim no)
+		(in_bom no)
+		(on_board yes)
+		(in_pos_files yes)
+		(dnp no)
+		(property "Reference" "JP3"
+			(at 210.566 105.156 0)
+			(show_name no)
+			(do_not_autoplace no)
+			(effects
+				(font
+					(size 1.27 1.27)
+				)
+			)
+		)
+		(property "Value" "SolderJumper_2_Open"
+			(at 210.566 102.616 0)
+			(show_name no)
+			(do_not_autoplace no)
+			(effects
+				(font
+					(size 1.27 1.27)
+				)
+			)
+		)
+		(property "Footprint" "Jumper:SolderJumper-2_P1.3mm_Open_TrianglePad1.0x1.5mm"
+			(at 210.82 107.95 0)
+			(hide yes)
+			(show_name no)
+			(do_not_autoplace no)
+			(effects
+				(font
+					(size 1.27 1.27)
+				)
+			)
+		)
+		(property "Datasheet" ""
+			(at 210.82 100.33 0)
+			(hide yes)
+			(show_name no)
+			(do_not_autoplace no)
+			(effects
+				(font
+					(size 1.27 1.27)
+				)
+			)
+		)
+		(property "Description" "Solder Jumper, 2-pole, open"
+			(at 210.82 102.87 0)
+			(hide yes)
+			(show_name no)
+			(do_not_autoplace no)
+			(effects
+				(font
+					(size 1.27 1.27)
+				)
+			)
+		)
+		(pin "1"
+		)
+		(pin "2"
+		)
+		(instances
+			(project "Undertray_Board"
+				(path "/85866aa8-1074-44e2-a4f8-fc50fec0cbab/74cdce65-3117-4a3b-a9a5-a5d0459f2000"
+					(reference "JP3")
+					(unit 1)
+				)

Commit message: button part change
Parts:
- SW2: value TL3301EF160QG -> PTS645SH43SMTR92 LFS
Changed lines of the file:
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@@
 			)
 		)
-		(property "Value" "TL3301EF160QG"
+		(property "Value" "PTS645SH43SMTR92 LFS"
 			(at 160.02 129.54 0)
 			(show_name no)

Commit message: button changes
Parts:
- SW2: footprint Button_Switch_SMD:SW_Push_1P1T_NO_CK_KSC6xxG -> Button_Switch_SMD:SW_Push_1P1T_NO_CK_KSC7xxJ
Changed lines of the file:
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@@
 			)
 		)
-		(property "Footprint" "Button_Switch_SMD:SW_Push_1P1T_NO_CK_KSC6xxG"
+		(property "Footprint" "Button_Switch_SMD:SW_Push_1P1T_NO_CK_KSC7xxJ"
 			(at 160.02 129.54 0)
 			(hide yes)
