File: 00-09_Projects/02_Sensors/02.06_CGGPS/hardware/CGGPS/CGGPS.kicad_sch (KiCad schematic)
At the start: 0 parts

Commit message: changes before schematic review
Parts:
- added H1, H2, H3, H4: MountingHole_Pad, MountingHole:MountingHole_3.2mm_M3_DIN965_Pad, symbol Mechanical:MountingHole_Pad
Connections:
- new net GND: H1.1, H2.1, H3.1, H4.1
Other:
- sheet Power_CAN renamed Power_CAN_IO
