File: 00-09_Projects/02_Sensors/02.06_CGGPS/hardware/CGGPS/GPS.kicad_sch (KiCad schematic)
At the start: 7 parts, among them J3 Conn_Coaxial, U2 ZED-F9P-02B

Commit message: wip
Parts:
- added D6: LED_RED, symbol Device:LED
- added D7: LED_BLUE, symbol Device:LED
- added R8: 33, symbol Device:R
- R2: value 33 -> 220
Connections:
- net GND: now also D6.1 (K), D7.1 (K)
- net GPS_TIMEPULSE: now reaches U2.53 (TIMEPULSE)
- net at C14.1, L1.1: now also U2.7 (VCC_RF); no longer R2.1
- net at R2.2: now also D6.2 (A); no longer U2.7 (VCC_RF)
- net GPS_VBACKUP: now reaches U2.36 (V_BCKP)
- net GEOFENCE_LED renamed GEOFENCE_STATUS
- net GEOFENCE_STATUS: now also R2.1
- net RTK_LED renamed RTK_STATUS
- net RTK_STATUS: now also R8.1
- new net: D7.2 (A), R8.2
- no-connect marks 21 -> 25
Other:
- note added: "650 Hz"
- note added: "GPS RF Receiver"
- note added: "GPS Status LEDs"
- note added: "GeoFence: Defined GPS boundary. Red when out of bounds. RTK: Phase measurements plus correction for cm accuracy. Solid when RTK correction, blinking when RTK correction is in progess, off when RTK is unable to correct."
- note added: "Need to decide if we need backup battery cell"
- moved on the sheet: C12, C13, C14, J3, L1, U2A, U2B

Commit message: wip
Parts:
- added C20: 1uF, symbol Device:C
- R10: renamed from R2; value 220 -> 330
- R11: renamed from R8; value 33 -> 330
- renumbered C14 to C17, C12 to C18, C13 to C19, D6 to D11, D7 to D12, U2 to U4
Connections:
- net GPS_VBACKUP is gone; now on net +3.3V: U4.36 (V_BCKP)
- net +3.3V: now also R11.1, C20.1; no longer U4.38 (V_USB)
- net GND: now also U4.32 (GND), U4.38 (V_USB), C20.2; no longer D12.1 (K)
- net RTK_STATUS: now also D12.1 (K); no longer R11.1
- net GPS_INT: no longer names the net of U4.51 (EXTINT)
- net SAFEBOOT_N: no longer names the net of U4.50 (SAFEBOOT_N)
- net USB+: no longer names the net of U4.40 (USB_DP)
- net USB-: no longer names the net of U4.39 (USB_DM)
- no-connect marks 25 -> 29

Commit message: changes before schematic review
Parts:
- C17: footprint (none) -> Capacitor_SMD:C_0402_1005Metric_Pad0.74x0.62mm_HandSolder
- C18, C19, C20: footprint (none) -> Capacitor_SMD:C_0603_1608Metric_Pad1.08x0.95mm_HandSolder
- D11, D12: footprint (none) -> Diode_SMD:D_0603_1608Metric_Pad1.05x0.95mm_HandSolder
- J5: renamed from J3; footprint (none) -> Connector_Coaxial:SMA_Molex_73251-1153_EdgeMount_Horizontal
- R10, R11: footprint (none) -> Resistor_SMD:R_0603_1608Metric_Pad0.98x0.95mm_HandSolder
- U4: footprint SMT_F9P-02B_UBL -> (none)
Other:
- moved on the sheet: C17, C18, C19, C20, D11, D12, J5, L1, R10, R11, U4A, U4B

Commit message: wip
Parts:
- L1: footprint (none) -> Inductor_SMD:L_0402_1005Metric_Pad0.77x0.64mm_HandSolder
- U4: footprint (none) -> CGGPS:SMT_F9P-02B_UBL
Other:
- note added: "LQW15AWR12J80D"
Changed lines of the file:
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@@
 		)
 	)
+	(text "LQW15AWR12J80D"
+		(exclude_from_sim no)
+		(at 29.464 55.626 90)
+		(effects
+			(font
+				(size 1.27 1.27)
+			)
+		)
+	)
 	(junction
 		(at 240.03 97.79)
@@
 			)
 		)
-		(property "Footprint" ""
+		(property "Footprint" "CGGPS:SMT_F9P-02B_UBL"
 			(at 187.96 44.45 0)
 			(hide yes)
@@
 			)
 		)
-		(property "Footprint" ""
+		(property "Footprint" "CGGPS:SMT_F9P-02B_UBL"
 			(at 55.88 45.72 0)
 			(hide yes)
@@
 			)
 		)
-		(property "Footprint" ""
+		(property "Footprint" "Inductor_SMD:L_0402_1005Metric_Pad0.77x0.64mm_HandSolder"
 			(at 33.02 54.61 0)
 			(hide yes)
