File: 00-09_Projects/02_Sensors/02.06_CGGPS/hardware/CGGPS/IMU.kicad_sch (KiCad schematic)
At the start: 12 parts, among them U3 BNO086, Y1 Crystal_GND24

Commit message: wip
Other:
- note added: "650 Hz"
Changed lines of the file:
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@@
+		)
+	)
+	(text "650 Hz"
+		(exclude_from_sim no)
+		(at 90.678 28.448 0)
+		(effects
+			(font
+				(size 1.27 1.27)
+			)
+			(justify left)
 		)
 	)

Commit message: wip
Parts:
- removed C10, C11: 12pF, symbol Device:C
- removed JP2, JP3, JP4, JP5: SolderJumper_2_Open, symbol Jumper:SolderJumper_2_Open
- removed Y1: Crystal_GND24, symbol Device:Crystal_GND24
- added R13, R14, R15, R16: 10k, symbol Device:R
- renumbered C9 to C21, C7 to C23, C8 to C25, R1 to R12, U3 to U5
Connections:
- net +3.3V: now also C23.1, C25.1, U5.10 (CLKSEL0), U5.28 (VDDIO), U5.3 (VDD), R13.1, R14.1, R15.1, R16.1; no longer U5.5 (PS1)
- net GND: now also U5.26 (XOUT32/CLKSEL1)
- net IMU_PS0/WAKE: now also R15.2
- net at U5.15 (ENV_SCL): now also R14.2
- net at U5.16 (ENV_SDA): now also R13.2
- new net: R16.2, U5.5 (PS1)
- no-connect marks 11 -> 10
Other:
- note removed: "BNO086 Crystal Oscillator"

Commit message: changes before schematic review
Parts:
- C21: footprint (none) -> Capacitor_SMD:C_0603_1608Metric_Pad1.08x0.95mm_HandSolder
- C22: renamed from C23; footprint (none) -> Capacitor_SMD:C_0603_1608Metric_Pad1.08x0.95mm_HandSolder
- C23: renamed from C25; footprint (none) -> Capacitor_SMD:C_0603_1608Metric_Pad1.08x0.95mm_HandSolder
- R12: renamed from R15; footprint (none) -> Resistor_SMD:R_0603_1608Metric_Pad0.98x0.95mm_HandSolder
- R13: renamed from R16; footprint (none) -> Resistor_SMD:R_0603_1608Metric_Pad0.98x0.95mm_HandSolder
- R14: renamed from R12; footprint (none) -> Resistor_SMD:R_0603_1608Metric_Pad0.98x0.95mm_HandSolder
- R15: renamed from R13; footprint (none) -> Resistor_SMD:R_0603_1608Metric_Pad0.98x0.95mm_HandSolder
- R16: renamed from R14; footprint (none) -> Resistor_SMD:R_0603_1608Metric_Pad0.98x0.95mm_HandSolder
- U5: footprint LGA-28_CEV -> (none)
Other:
- moved on the sheet: C21, C22, C23, R12, R13, R14, R15, R16, U5

Commit message: wip
Parts:
- U5: footprint (none) -> CGGPS:BN0086_1_LGA-28_CEV
Changed lines of the file:
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@@
 			)
 		)
-		(property "Footprint" ""
+		(property "Footprint" "CGGPS:BN0086_1_LGA-28_CEV"
 			(at 87.63 55.88 0)
 			(hide yes)
