File: 00-09_Projects/02_Sensors/02.06_CGGPS/hardware/CGGPS/MCU.kicad_sch (KiCad schematic)
At the start: 9 parts, among them U1 STM32F302C8Tx

Commit message: wip
Parts:
- added C21, C22: 0.1uF, symbol Device:C
- added C23: 1uF, symbol Device:C
- added D10: ACPDQC3V3T-HF, symbol Device:D_Schottky
- added D11: LED_AMBER, symbol Device:LED
- added D8: D_Schottky, symbol Device:D_Schottky
- added D9: LED_RED, symbol Device:LED
- added R10, R9: 220, symbol Device:R
- added R11: 47k, symbol Device:R
- added SW1: SW_Push, symbol Switch:SW_Push
- added SW2: SW_Nidec_CAS-120A1, Button_Switch_SMD:Nidec_Copal_CAS-120A, symbol Switch:SW_Nidec_CAS-120A1
- added U6: 74AUC2G32, symbol 74xGxx:74AUC2G32
Connections:
- net +3.3V: now also D9.2 (A), SW2.3 (A), U6.8 (VCC)
- net BOOT0: now also R10.1, U6.7
- net CANRX: now also U1.45 (PB8)
- net CANTX: now also U1.46 (PB9)
- net GND: now also C21.2, C22.2, C23.2, D10.2 (A), D11.1 (K), D8.2 (A), SW1.2, SW2.1 (C), SW2.4 (MP), SW2.5 (MP), SW2.6 (MP), U6.4 (GND)
- net NRST: now also C21.1, D8.1 (K), R9.2, SW1.1
- net USART2_TX: now reaches U1.12 (PA2)
- net USART2_RX: now reaches U1.13 (PA3)
- net BOOT0_TRIG: now reaches U1.18 (PB0)
- net BOOT0_TRIG: now also R11.1
- net IMU_NRST: now reaches U1.19 (PB1)
- net IMU_PS0/WAKE: now reaches U1.20 (PB2)
- net RTK_STATUS: now reaches U1.21 (PB10)
- net GEOFENCE_STATUS: now reaches U1.22 (PB11)
- net GPS_CS: now reaches U1.25 (PB12)
- net GPS_SCLK: now reaches U1.26 (PB13)
- net GPS_MISO: now reaches U1.27 (PB14)
- net GPS_MOSI: now reaches U1.28 (PB15)
- net GPS_TXD2: now reaches U1.30 (PA9)
- net GPS_RXD2: now reaches U1.31 (PA10)
- net IMU_SCLK: now reaches U1.39 (PB3)
- net IMU_MISO: now reaches U1.40 (PB4)
- net IMU_MOSI: now reaches U1.41 (PB5)
- net IMU_CS: now reaches U1.42 (PB6)
- net CAN_SLEEP: now reaches U1.43 (PB7)
- new net: C22.1, R11.2, U6.2
- new net: D9.1 (K), R9.1
- new net: D11.2 (A), R10.2
- new net BOOT0_SW: C23.1, D10.1 (K), SW2.2 (B), U6.1
- no-connect marks 0 -> 3
Other:
- note added: "BOOT0 Switch"
- note added: "MCU Power"
- note added: "Reset Button"
- note added: "STM32F302C8T6"

Commit message: wip
Parts:
- removed C22: 0.1uF, symbol Device:C
- removed D11: LED_AMBER, symbol Device:LED
- removed R10: 220, symbol Device:R
- removed R11: 47k, symbol Device:R
- removed U6: 74AUC2G32, symbol 74xGxx:74AUC2G32
- added C7, C8: 12pF, symbol Device:C
- added D9: LED_AMBER, symbol Device:LED
- added J4: SHF-107-01-L-D-SM, SHF-107-01-L-D-SM:SAMTEC_SHF-107-01-L-D-SM, symbol CGGPS:SHF-107-01-L-D-SM
- added R7, R9: 220, symbol Device:R
- added Y1: Crystal_GND24, symbol Device:Crystal_GND24
- D8: value D_Schottky -> ACPDQC3V3T-HF
- renumbered C6 to C10, C21 to C11, C2 to C12, C5 to C13, C3 to C14, C4 to C15, C23 to C16, C1 to C9, D9 to D7, R9 to R8, U1 to U3
Connections:
- net BOOT0_SW is gone; now on net BOOT0: C16.1, D10.1 (K), SW2.2 (B)
- net +3.3V: now also J4.03
- net BOOT0: now also R9.1
- net GND: now also C7.2, C8.2, D9.1 (K), J4.05, J4.07, J4.11, Y1.2 (G), Y1.4 (G)
- net GPS_RXD2: now also U3.30 (PA9); no longer U3.31 (PA10)
- net GPS_TXD2: now also U3.31 (PA10); no longer U3.30 (PA9)
- net NRST: now also J4.12
- net RCC_OSC_IN: now also C7.1, Y1.1
- net RCC_OSC_OUT: now also R7.2
- net SWCLK: now also J4.06
- net SWDIO: now also J4.04
- net BOOT0_TRIG renamed IMU_H_INTN
- new net: D9.2 (A), R9.2
- new net: C8.1, R7.1, Y1.3
- no-connect marks 3 -> 8
Other:
- note added: "Debug Connector"
- note added: "MCU Oscillator Crystal"
- moved on the sheet: C11, C16, D10, D7, D8, R8, SW1, SW2

Commit message: changes before schematic review
Parts:
- C10, C11, C12, C13, C14, C16, C9: footprint (none) -> Capacitor_SMD:C_0603_1608Metric_Pad1.08x0.95mm_HandSolder
- C15: footprint (none) -> Capacitor_SMD:C_0805_2012Metric_Pad1.18x1.45mm_HandSolder
- C7, C8: footprint (none) -> Capacitor_SMD:C_0402_1005Metric_Pad0.74x0.62mm_HandSolder
- D7, D9: footprint (none) -> Diode_SMD:D_0603_1608Metric_Pad1.05x0.95mm_HandSolder
- JP1: footprint (none) -> Jumper:SolderJumper-2_P1.3mm_Open_TrianglePad1.0x1.5mm
- R7: footprint (none) -> Resistor_SMD:R_0603_1608Metric_Pad0.98x0.95mm_HandSolder
- R8, R9: value 220 -> 330; footprint (none) -> Resistor_SMD:R_0603_1608Metric_Pad0.98x0.95mm_HandSolder
Connections:
- net GPS_TIMEPULSE: now reaches U3.29 (PA8)
- no-connect marks 8 -> 17
Other:
- moved on the sheet: C10, C11, C12, C13, C14, C15, C16, C9, D10, D7, D8, D9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

Commit message: wip
Parts:
- D10, D8: footprint (none) -> Diode_SMD:D_0402_1005Metric_Pad0.77x0.64mm_HandSolder
- SW2: footprint Button_Switch_SMD:Nidec_Copal_CAS-120A -> (none)
Changed lines of the file:
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@@
 			)
 		)
-		(property "Footprint" "Button_Switch_SMD:Nidec_Copal_CAS-120A"
+		(property "Footprint" ""
 			(at 233.68 46.99 0)
 			(hide yes)
@@
 			)
 		)
-		(property "Footprint" ""
+		(property "Footprint" "Diode_SMD:D_0402_1005Metric_Pad0.77x0.64mm_HandSolder"
 			(at 220.98 46.99 0)
 			(hide yes)
@@
 			)
 		)
-		(property "Footprint" ""
+		(property "Footprint" "Diode_SMD:D_0402_1005Metric_Pad0.77x0.64mm_HandSolder"
 			(at 135.89 116.84 0)
 			(hide yes)
