File: 00-09_Projects/02_Sensors/02.06_CGGPS/hardware/CGGPS/Power_CAN.kicad_sch (KiCad schematic)
At the start: 22 parts, among them J1 USB_C_Receptacle_USB2.0_14P, J4 Conn_01x04_Socket, U4 SN65HVD230, U5 AP2210K-3.3TRG1

Commit message: wip
Parts:
- R7: value R -> 220
Connections:
- net +3.3V: now also C20.1, R7.1, U5.5 (VOUT)
- net GND: now also C20.2, D5.1 (K)
Other:
- note added: "+5V Protection"
- note added: "+5V to +3.3V LDO"
- moved on the sheet: C17, C18, C19, C20, D2, D3, D4, D5, F1, J4, R6, R7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

Commit message: wip
Parts:
- added F2: 200mA, symbol Device:Fuse
- added R3: 120, symbol Device:R
- F1: value 750mA -> 200mA
- R2: renamed from R6; value 220 -> 330
- R6: renamed from R7; value 220 -> 330
- renumbered C15 to C1, C18 to C2, C16 to C3, C17 to C4, C19 to C5, C20 to C6, D2 to D1, D3 to D2, CR1 to D3, D1 to D5, D5 to D6, J4 to J2, R5 to R1, R3 to R4, R4 to R5, U4 to U1, U5 to U2
Connections:
- net +3.3V: now also F2.2; no longer U2.5 (VOUT)
- net CANH: now also R3.1
- net CANL: now also R3.2
- net USB-: now reaches D5.2 (I/O1), J1.A7 (D-), J1.B7 (D-)
- net USB+: now reaches D5.3 (I/O2), J1.A6 (D+), J1.B6 (D+)
- new net: F2.1, U2.5 (VOUT)

Commit message: changes before schematic review
Parts:
- added J2: Conn_01x06_Pin, Connector_PinHeader_2.54mm:PinHeader_1x06_P2.54mm_Vertical, symbol Connector:Conn_01x06_Pin
- C1, C3, C4, C5: footprint (none) -> Capacitor_SMD:C_0603_1608Metric_Pad1.08x0.95mm_HandSolder
- C2, C6: footprint (none) -> Capacitor_SMD:C_0805_2012Metric_Pad1.18x1.45mm_HandSolder
- D3: footprint SOT-23_DBZ_TEX -> (none)
- D4: footprint (none) -> Diode_SMD:D_0603_1608Metric_Pad1.05x0.95mm_HandSolder
- D6: value LED -> LED_GREEN; footprint (none) -> Diode_SMD:D_0603_1608Metric_Pad1.05x0.95mm_HandSolder
- J1: footprint (none) -> Connector_USB:USB_C_Receptacle_HRO_TYPE-C-31-M-12
- R1, R2, R4, R5, R6: footprint (none) -> Resistor_SMD:R_0603_1608Metric_Pad0.98x0.95mm_HandSolder
- R3: footprint (none) -> Resistor_SMD:R_0603_1608Metric_Pad0.98x0.95mm_HandSolder; now not fitted
- U2: footprint SOT-23-5_DIO -> LHR:SOT-23-5_DIO
- renumbered J2 to J3
Connections:
- net +5V: now also U2.1 (VIN), U2.3 (EN)
- net CANH: now also J2.1 (Pin_1)
- net CANL: now also J2.2 (Pin_2)
- net GND: now also J2.3 (Pin_3), J2.4 (Pin_4)
- new net USART2_RX: J2.6 (Pin_6)
- new net USART2_TX: J2.5 (Pin_5)
Other:
- note added: "Debug header pins"
- moved on the sheet: C1, C3, C4, C5, C6, D5, D6, F2, J1, J3, R4, R5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

Commit message: wip
Parts:
- D1: value RB520S30T5G -> SDM20U30-7; footprint Diode_THT:D_DO-35_SOD27_P7.62mm_Horizontal -> Diode_SMD:D_SOD-523
- D3: footprint (none) -> Package_TO_SOT_SMD:SOT-23-3
Changed lines of the file:
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@@
 			)
 		)
-		(property "Value" "RB520S30T5G"
+		(property "Value" "SDM20U30-7"
 			(at 36.83 104.14 0)
 			(show_name no)
@@
 			)
 		)
-		(property "Footprint" "Diode_THT:D_DO-35_SOD27_P7.62mm_Horizontal"
+		(property "Footprint" "Diode_SMD:D_SOD-523"
 			(at 36.83 103.505 0)
 			(hide yes)
@@
 			)
 		)
-		(property "Footprint" ""
+		(property "Footprint" "Package_TO_SOT_SMD:SOT-23-3"
 			(at 80.01 50.8 0)
 			(hide yes)

Commit message: pre schematic review changes
Parts:
- F1, F2: value 200mA -> 250mA; footprint (none) -> Fuse:Fuse_1206_3216Metric_Pad1.42x1.75mm_HandSolder
Changed lines of the file:
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@@
 			)
 		)
-		(property "Value" "200mA"
+		(property "Value" "250mA"
 			(at 195.58 105.41 90)
 			(show_name no)
@@
 			)
 		)
-		(property "Footprint" ""
+		(property "Footprint" "Fuse:Fuse_1206_3216Metric_Pad1.42x1.75mm_HandSolder"
 			(at 195.58 110.998 90)
 			(hide yes)
@@
 			)
 		)
-		(property "Value" "200mA"
+		(property "Value" "250mA"
 			(at 48.26 104.14 90)
 			(show_name no)
@@
 			)
 		)
-		(property "Footprint" ""
+		(property "Footprint" "Fuse:Fuse_1206_3216Metric_Pad1.42x1.75mm_HandSolder"
 			(at 48.26 109.728 90)
 			(hide yes)
